Commit message: Prepare GraspQP open-source release
- Migrate grasp-synthesis code, hands, and IsaacLab integration from the
  internal repo; drop copyright-restricted assets (XHand, HOI, dex3) and the
  dex_retargeting dependency.
- Add ETH Zurich OSS licensing (LICENSE, NOTICE, AUTHORS, SPDX headers).
- Add slim (WARP) and full (TorchSDF) Docker images; default SDF backend WARP.
- Add test suite: grasp-optimization smoke test, pytorch3d-compat, hand
  registry, transforms/FK, plus a bundled dummy_sphere asset.
- Fix gendexgrasp energy selection, pin pytorch_kinematics, add pycollada.
- Google-style docstrings across core/hands/metrics/utils and improved docs.

File: graspqp/assets/shadow_hand/shadow_hand.urdf (robot description, URDF)
Before this commit: robot shadow_hand, 27 links, 26 joints
Links:
- added link robot0_fftip
- added link robot0_lftip
- added link robot0_mftip
- added link robot0_palm_center
- added link robot0_rftip
- added link robot0_thtip
Joints:
- added joint fftip: type fixed, parent robot0_ffdistal, child robot0_fftip, origin xyz=0. 0. 0.03 rpy=0. 0. 0.
- added joint lftip: type fixed, parent robot0_lfdistal, child robot0_lftip, origin xyz=0. 0. 0.03 rpy=0. 0. 0.
- added joint mftip: type fixed, parent robot0_mfdistal, child robot0_mftip, origin xyz=0. 0. 0.03 rpy=0. 0. 0.
- added joint palm_center: type fixed, parent robot0_palm, child robot0_palm_center, origin xyz=-0.0 0.0 0.035 rpy=0. 0. 0.
- added joint rftip: type fixed, parent robot0_rfdistal, child robot0_rftip, origin xyz=0. 0. 0.03 rpy=0. 0. 0.
- added joint thtip: type fixed, parent robot0_thdistal, child robot0_thtip, origin xyz=0. 0. 0.038 rpy=0. 0. 0.
- joint robot0_WRJ0: type revolute -> fixed
- joint robot0_WRJ1: type revolute -> fixed
